Commit message: should be good to go diff --git a/README.md b/README.md index e4cf169..e554b3f 100644 --- a/README.md +++ b/README.md @@ -1,5 +1,5 @@ -# Mila Slider +# Mila Pusher
-This is a fork from Poppy Ergo Jr but modified for a 2-DoF sliding configuration.
+This is a fork from Poppy Ergo Jr but modified for a 3-DoF sliding configuration.

 More documentation to follow.
\ No newline at end of file
diff --git a/software/mila_pusher/__init__.py b/software/mila_pusher/__init__.py
new file mode 100644
index 0000000..36cb51d
--- /dev/null
+++ b/software/mila_pusher/__init__.py
@@ -0,0 +1 @@
+from .mila_pusher import MilaPusher
\ No newline at end of file
diff --git a/software/mila_slider/configuration/mila_slider.json b/software/mila_pusher/configuration/mila_slider.json
similarity index 70%
rename from software/mila_slider/configuration/mila_slider.json
rename to software/mila_pusher/configuration/mila_slider.json
index 2abe364..f68aa15 100644
--- a/software/mila_slider/configuration/mila_slider.json
+++ b/software/mila_pusher/configuration/mila_slider.json
@@ -13,7 +13,8 @@
   "motorgroups": {
     "base": [
       "m1",
-      "m2"
+      "m2",
+      "m3"
     ]
   },
   "motors": {
@@ -22,8 +23,8 @@
       "type": "XL-320",
       "id": 1,
       "angle_limit": [
-        -45.0,
-        45.0
+        -90.0,
+        90.0
       ],
       "orientation": "direct"
     },
@@ -32,18 +33,23 @@
       "type": "XL-320",
       "id": 2,
       "angle_limit": [
-        45.0,
-        135.0
+        -90.0,
+        90.0
+      ],
+      "orientation": "direct"
+    },
+    "m3": {
+      "offset": 0.0,
+      "type": "XL-320",
+      "id": 2,
+      "angle_limit": [
+        -90.0,
+        90.0
       ],
       "orientation": "direct"
     }
   },
   "sensors": {
-     "camera": {
-      "type": "OpenCVCamera",
-      "index": -1,
-      "fps": 100.0,
-      "resolution": [640, 480]
-    }
+
   }
 }
diff --git a/software/mila_slider/mila_slider.py b/software/mila_pusher/mila_pusher.py
similarity index 93%
rename from software/mila_slider/mila_slider.py
rename to software/mila_pusher/mila_pusher.py
index 901cea5..fcd82ea 100644
--- a/software/mila_slider/mila_slider.py
+++ b/software/mila_pusher/mila_pusher.py
@@ -5,7 +5,7 @@ from pypot.creatures import AbstractPoppyCreature
 from pypot.creatures.ik import IKChain

-class MilaSlider(AbstractPoppyCreature):
+class MilaPusher(AbstractPoppyCreature):
     @classmethod
     def setup(cls, robot):
         robot._primitive_manager._filter = partial(sum, axis=0)
diff --git a/software/mila_slider/mila_slider.urdf b/software/mila_pusher/mila_pusher.urdf
similarity index 70%
rename from software/mila_slider/mila_slider.urdf
rename to software/mila_pusher/mila_pusher.urdf
index 3e018cf..d273e4d 100644
--- a/software/mila_slider/mila_slider.urdf
+++ b/software/mila_pusher/mila_pusher.urdf
@@ -145,5 +145,58 @@
       link="section_1" />
     <axis
       xyz="-1 0 0" />
+  </joint>
+   <link
+    name="section_2">
+    <inertial>
+      <origin
+        xyz="-0.000168296047337745 0.013441283142678 -3.36410230095056E-09"
+        rpy="0 0 0" />
+      <mass
+        value="0.0201321844066136" />
+      <inertia
+        ixx="6.51960684491032E-06"
+        ixy="-5.35361387413197E-07"
+        ixz="-5.67167110473808E-13"
+        iyy="2.37206686086462E-06"
+        iyz="-1.07202400036876E-12"
+        izz="7.46616268702629E-06" />
+    </inertial>
+    <visual>
+      <origin
+        xyz="0 0 0"
+        rpy="0 0 0" />
+      <geometry>
+        <mesh
+          filename="package://PoppyErgoJr/meshes/section_1.STL" />
+      </geometry>
+      <material
+        name="">
+        <color
+          rgba="0.752941176470588 0.752941176470588 0.752941176470588 1" />
+      </material>
+    </visual>
+    <collision>
+      <origin
+        xyz="0 0 0"
+        rpy="0 0 0" />
+      <geometry>
+        <mesh
+          filename="package://PoppyErgoJr/meshes/section_1.STL" />
+      </geometry>
+    </collision>
+  </link>
+  <joint
+    name="m3"
+    type="continuous">
+    <origin
+      xyz="0 0 0.0240006783879033"
+      rpy="1.5707963267949 0 0" />
+    <parent
+      link="section_1" />
+    <child
+      link="section_2" />
+    <axis
+      xyz="-1 0 0" />
   </joint>
 </robot>
diff --git a/software/mila_slider/__init__.py b/software/mila_slider/__init__.py
deleted file mode 100644
index c37b070..0000000
--- a/software/mila_slider/__init__.py
+++ /dev/null
@@ -1 +0,0 @@
-from .mila_slider import MilaSlider
\ No newline at end of file
diff --git a/software/setup.py b/software/setup.py
index 208e2ac..92caf11 100644
--- a/software/setup.py
+++ b/software/setup.py
@@ -1,6 +1,6 @@
 from setuptools import setup

-setup(name='mila-slider',
+setup(name='mila-pusher',
       version="1.0",
       install_requires=[
           'pypot >= 3',

File: software/mila_pusher/mila_pusher.urdf (robot description, URDF)
Before this commit: robot PoppyErgoJr, 3 links, 2 joints
Links:
- added link section_2, mass 0.0201321844066136; collision mesh filename=package://PoppyErgoJr/meshes/section_1.STL; visual mesh filename=package://PoppyErgoJr/meshes/section_1.STL
Joints:
- added joint m3: type continuous, parent section_1, child section_2, origin xyz=0 0 0.0240006783879033 rpy=1.5707963267949 0 0, axis -1 0 0
